File: pcb/pcb.kicad_sch (KiCad schematic)
At the start: 101 parts, among them J1 I2C, J2 HR911105A, J3 USB_C_Receptacle_USB2.0, J4 GPS, J5 DNP, Q1 BC817, Q2 WPM2015-3_TR, Q3 BC817, Q4 BC817, Q5 BC817, SW1 DNP, SW2 DNP, U1 ESP32-WROOM-32D, U2 LAN8710A, U3 ADXL355, U4 MIC5219-3.3YM5, U5 74LVC1G17, U6 CP2102N-Axx-xQFN24

Commit message: Fixed UART RX/TX lines
Connections:
- net RXD0: now also U6.21 (TXD); no longer U6.20 (RXD)
- net TXD0: now also U6.20 (RXD); no longer U6.21 (TXD)
Changed lines of the file:
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@@
   (junction (at 381 96.52) (diameter 0) (color 0 0 0 0))
   (junction (at 391.16 99.06) (diameter 0) (color 0 0 0 0))
+  (no_connect (at 153.67 226.06))
+  (no_connect (at 190.5 82.55))
+  (no_connect (at 252.73 66.04))
+  (no_connect (at 190.5 72.39))
+  (no_connect (at 113.03 208.28))
   (no_connect (at 252.73 101.6))
+  (no_connect (at 190.5 69.85))
+  (no_connect (at 190.5 54.61))
+  (no_connect (at 113.03 220.98))
+  (no_connect (at 252.73 93.98))
+  (no_connect (at 113.03 193.04))
+  (no_connect (at 252.73 96.52))
+  (no_connect (at 190.5 85.09))
   (no_connect (at 57.15 66.04))
-  (no_connect (at 190.5 72.39))
-  (no_connect (at 190.5 69.85))
-  (no_connect (at 190.5 85.09))
-  (no_connect (at 252.73 66.04))
   (no_connect (at 190.5 62.23))
+  (no_connect (at 113.03 241.3))
+  (no_connect (at 190.5 64.77))
+  (no_connect (at 252.73 63.5))
+  (no_connect (at 373.38 101.6))
+  (no_connect (at 314.96 177.8))
+  (no_connect (at 57.15 63.5))
+  (no_connect (at 252.73 99.06))
   (no_connect (at 190.5 57.15))
-  (no_connect (at 113.03 193.04))
-  (no_connect (at 113.03 208.28))
-  (no_connect (at 252.73 99.06))
-  (no_connect (at 252.73 93.98))
-  (no_connect (at 373.38 101.6))
-  (no_connect (at 113.03 220.98))
-  (no_connect (at 252.73 63.5))
-  (no_connect (at 190.5 64.77))
-  (no_connect (at 153.67 226.06))
-  (no_connect (at 314.96 177.8))
-  (no_connect (at 190.5 82.55))
-  (no_connect (at 113.03 241.3))
-  (no_connect (at 252.73 96.52))
-  (no_connect (at 57.15 63.5))
-  (no_connect (at 190.5 54.61))
   (bus_entry (at 198.12 46.99) (size 2.54 -2.54)
     (stroke (width 0.1524) (type solid) (color 0 0 0 0))
@@
     (stroke (width 0) (type solid) (color 0 0 0 0))
   )
-  (wire (pts (xy 190.5 46.99) (xy 198.12 46.99))
+  (wire (pts (xy 190.5 49.53) (xy 198.12 49.53))
     (stroke (width 0) (type solid) (color 0 0 0 0))
   )
@@
     (stroke (width 0) (type solid) (color 0 0 0 0))
   )
-  (wire (pts (xy 198.12 49.53) (xy 190.5 49.53))
+  (wire (pts (xy 198.12 46.99) (xy 190.5 46.99))
     (stroke (width 0) (type solid) (color 0 0 0 0))
   )
@@
     (stroke (width 0) (type solid) (color 0 0 0 0))
   )
-  (bus (pts (xy 306.07 64.77) (xy 306.07 66.04))
-    (stroke (width 0) (type solid) (color 0 0 0 0))
-  )
-  (bus (pts (xy 306.07 66.04) (xy 306.07 73.66))
+  (bus (pts (xy 306.07 64.77) (xy 306.07 71.12))
+    (stroke (width 0) (type solid) (color 0 0 0 0))
+  )
+  (bus (pts (xy 306.07 71.12) (xy 306.07 73.66))
     (stroke (width 0) (type solid) (color 0 0 0 0))
   )
@@
     (stroke (width 0) (type solid) (color 0 0 0 0))
   )
-  (bus (pts (xy 316.23 91.44) (xy 316.23 93.98))
-    (stroke (width 0) (type solid) (color 0 0 0 0))
-  )
-  (bus (pts (xy 316.23 93.98) (xy 316.23 99.06))
-    (stroke (width 0) (type solid) (color 0 0 0 0))
-  )
-  (bus (pts (xy 316.23 99.06) (xy 316.23 104.14))
-    (stroke (width 0) (type solid) (color 0 0 0 0))
-  )
-  (bus (pts (xy 316.23 104.14) (xy 316.23 109.22))
-    (stroke (width 0) (type solid) (color 0 0 0 0))
-  )
-  (bus (pts (xy 316.23 109.22) (xy 316.23 114.3))
+  (bus (pts (xy 316.23 91.44) (xy 316.23 96.52))
+    (stroke (width 0) (type solid) (color 0 0 0 0))
+  )
+  (bus (pts (xy 316.23 96.52) (xy 316.23 101.6))
+    (stroke (width 0) (type solid) (color 0 0 0 0))
+  )
+  (bus (pts (xy 316.23 101.6) (xy 316.23 106.68))
+    (stroke (width 0) (type solid) (color 0 0 0 0))
+  )
+  (bus (pts (xy 316.23 106.68) (xy 316.23 114.3))
     (stroke (width 0) (type solid) (color 0 0 0 0))
   )
@@
     (effects (font (size 0.762 0.762)) (justify left bottom))
   )
-  (label "TXD0" (at 198.12 46.99 180)
-    (effects (font (size 1.27 1.27)) (justify right bottom))
-  )
-  (label "RXD0" (at 198.12 49.53 180)
-    (effects (font (size 1.27 1.27)) (justify right bottom))
-  )
+  (label "RXD0" (at 198.12 46.99 180)
+    (effects (font (size 1.27 1.27)) (justify right bottom))
+  )
+  (label "TXD0" (at 198.12 49.53 180)
+    (effects (font (size 1.27 1.27)) (justify right bottom))
+  )
